File: gvpsimm.sch (KiCad schematic (older format))
At the start: 18 parts, among them J1 SIMM64_EDGE, U1 HM514400_alt, U2 HM514400_alt, U3 HM514400_alt, U4 HM514400_alt, U5 HM514400_alt, U6 HM514400_alt, U7 HM514400_alt, U8 HM514400_alt

Commit message: 16MB study
Parts:
- added U?: DRAM-4Mx4-SOP-24, stdpads:SOP-24-26-300mil, symbol GW_RAM:DRAM-4Mx4-SOP-24
- J1: symbol memory:SIMM64_EDGE -> gvpsimm-rescue:SIMM64_EDGE-memory
- U1, U2, U3, U4, U5, U6, U7, U8: symbol memory:HM514400_alt -> gvpsimm-rescue:HM514400_alt-memory
Changed lines of the file:
@@
 EESchema Schematic File Version 4
-LIBS:gvpsimm-cache
-EELAYER 29 0
+EELAYER 30 0
 EELAYER END
 $Descr A4 11693 8268
@@
 $EndDescr
 $Comp
-L memory:SIMM64_EDGE J1
+L gvpsimm-rescue:SIMM64_EDGE-memory J1
 U 1 1 5D395819
 P 2350 2000
@@
 DQ0
 $Comp
-L memory:HM514400_alt U1
+L gvpsimm-rescue:HM514400_alt-memory U1
 U 1 1 5D3B5A01
 P 4700 1250
@@
 	6800 1700 7100 1700
 $Comp
-L memory:HM514400_alt U2
+L gvpsimm-rescue:HM514400_alt-memory U2
 U 1 1 5D3B6C79
 P 6350 1250
@@
 	8450 1700 8750 1700
 $Comp
-L memory:HM514400_alt U3
+L gvpsimm-rescue:HM514400_alt-memory U3
 U 1 1 5D3C02FF
 P 8000 1250
@@
 	10100 1700 10400 1700
 $Comp
-L memory:HM514400_alt U4
+L gvpsimm-rescue:HM514400_alt-memory U4
 U 1 1 5D3C0330
 P 9650 1250
@@
 	5150 4500 5450 4500
 $Comp
-L memory:HM514400_alt U5
+L gvpsimm-rescue:HM514400_alt-memory U5
 U 1 1 5D3D1685
 P 4700 4050
@@
 	6800 4500 7100 4500
 $Comp
-L memory:HM514400_alt U6
+L gvpsimm-rescue:HM514400_alt-memory U6
 U 1 1 5D3D16B6
 P 6350 4050
@@
 	8450 4500 8750 4500
 $Comp
-L memory:HM514400_alt U7
+L gvpsimm-rescue:HM514400_alt-memory U7
 U 1 1 5D3D16E7
 P 8000 4050
@@
 	10100 4500 10400 4500
 $Comp
-L memory:HM514400_alt U8
+L gvpsimm-rescue:HM514400_alt-memory U8
 U 1 1 5D3D1718
 P 9650 4050
@@
 Text Notes 7150 6950 0    50   ~ 0
 BY @TubeTimeUS\n
+$Comp
+L GW_RAM:DRAM-4Mx4-SOP-24 U?
+U 1 1 5EBDE0C9
+P 12450 2250
+F 0 "U?" H 12450 3017 50  0000 C CNN
+F 1 "DRAM-4Mx4-SOP-24" H 12450 2926 50  0000 C CNN
+F 2 "stdpads:SOP-24-26-300mil" H 12450 1600 50  0001 C CNN
+F 3 "https://shop.micross.com/pdf/AS4C4M4.pdf" H 12450 1650 50  0001 C CNN
+	1    12450 2250
+	1    0    0    -1
+$EndComp
 $EndSCHEMATC
